Commit message: fix(rihibot): replaced gazebo imu plugin #1000
replaced the libgazebo_ros_imu plugin with the libgazebo_ros_imu_sensor
plugin to get the measurements relative to imu_link instead of
wrist_3_link

File: atom_examples/rihibot/rihibot_description/urdf/imu.urdf.xacro (robot description, xacro)
@@ -36,31 +36,49 @@
 			</inertial>
 		</link>
-		<gazebo>
-			<plugin name="imu_plugin" filename="libgazebo_ros_imu.so">
-			<alwaysOn>true</alwaysOn>
-			<bodyName>imu_link</bodyName>
-			<frameName>imu_link</frameName>
-			<topicName>imu</topicName>
-			<serviceName>imu_service</serviceName>
-			<gaussianNoise>0.0</gaussianNoise>
-			<updateRate>200</updateRate>
-			<imu>
-				<noise>
-				<type>gaussian</type>
-				<rate>
-					<mean>0.0</mean>
-					<stddev>2e-4</stddev>
-					<bias_mean>0.0000075</bias_mean>
-					<bias_stddev>0.0000008</bias_stddev>
-				</rate>
-				<accel>
-					<mean>0.0</mean>
-					<stddev>1.7e-2</stddev>
-					<bias_mean>0.1</bias_mean>
-					<bias_stddev>0.001</bias_stddev>
-				</accel>
-				</noise>
-			</imu>
+		<gazebo reference="${prefix}_link">
+			<!-- <plugin name="imu_plugin" filename="libgazebo_ros_imu.so"> -->
+				<!-- <alwaysOn>true</alwaysOn> -->
+				<!-- <bodyName>imu_link</bodyName> -->
+				<!-- <frameName>imu_link</frameName> -->
+				<!-- <topicName>imu</topicName> -->
+				<!-- <serviceName>imu_service</serviceName> -->
+				<!-- <gaussianNoise>0.0</gaussianNoise> -->
+				<!-- <updateRate>200</updateRate> -->
+				<!-- <imu> -->
+					<!-- <noise> -->
+					<!-- <type>gaussian</type> -->
+					<!-- <rate> -->
+						<!-- <mean>0.0</mean> -->
+						<!-- <stddev>2e-4</stddev> -->
+						<!-- <bias_mean>0.0000075</bias_mean> -->
+						<!-- <bias_stddev>0.0000008</bias_stddev> -->
+					<!-- </rate> -->
+					<!-- <accel> -->
+						<!-- <mean>0.0</mean> -->
+						<!-- <stddev>1.7e-2</stddev> -->
+						<!-- <bias_mean>0.1</bias_mean> -->
+						<!-- <bias_stddev>0.001</bias_stddev> -->
+					<!-- </accel> -->
+					<!-- </noise> -->
+				<!-- </imu> -->
+			<!-- </plugin> -->
+    	<gravity>true</gravity>
+    	<sensor name="imu_sensor" type="imu">
+			<always_on>true</always_on>
+			<update_rate>100</update_rate>
+			<visualize>true</visualize>
+			<topic>__default_topic__</topic>
+				<plugin filename="libgazebo_ros_imu_sensor.so" name="imu_plugin">
+				<topicName>imu</topicName>
+				<bodyName>imu_link</bodyName>
+				<updateRateHZ>200.0</updateRateHZ>
+				<gaussianNoise>0.0</gaussianNoise>
+				<xyzOffset>0 0 0</xyzOffset>
+				<rpyOffset>0 0 0</rpyOffset>
+				<frameName>imu_link</frameName>
+				<initialOrientationAsReference>false</initialOrientationAsReference>
 			</plugin>
+			<pose>0 0 0 0 0 0</pose>
+    	</sensor>
 		</gazebo>
 </xacro:macro>

File: atom_examples/rihibot/rihibot_description/urdf/robot.urdf.xacro (robot description, xacro)
@@ -81,5 +81,5 @@
     <!-- IMU -->
     <xacro:imu parent="flange" prefix="imu" color_gazebo="Red">
-        <origin xyz="0.01 0 0" rpy="0 0 0" />
+        <origin xyz="10 0 0" rpy="0 0 0" />
         <color_rgb_rviz>
             <material name="red">
