Commit message: feat(rihibot): added imu and respective plugin #1000
added an IMU to the rihibot system, using the libgazebo_ros_imu.so
plugin

File: atom_examples/rihibot/rihibot_description/urdf/robot.urdf.xacro (robot description, xacro)
@@ -40,4 +40,5 @@
     <!-- Sensors-->
     <xacro:include filename="$(find rihibot_description)/urdf/rgb_camera.urdf.xacro" />
+    <xacro:include filename="$(find rihibot_description)/urdf/imu.urdf.xacro"/>
     <!-- Manipulator-->
     <xacro:include filename="$(find ur_gazebo)/urdf/ur_macro.xacro"/>
@@ -78,3 +79,12 @@
         </color_rgb_rviz>
     </xacro:rgb_camera>
+    <!-- IMU -->
+    <xacro:imu parent="flange" prefix="imu" color_gazebo="Red">
+        <origin xyz="0.01 0 0" rpy="0 0 0" />
+        <color_rgb_rviz>
+            <material name="red">
+                <color rgba="0.9 0 0 1"/>
+            </material>
+        </color_rgb_rviz>
+    </xacro:imu>
 </robot>

Commit message: fix(rihibot): fixed IMU pose on the end-effector #1000

File: atom_examples/rihibot/rihibot_description/urdf/robot.urdf.xacro (robot description, xacro)
@@ -81,5 +81,5 @@
     <!-- IMU -->
     <xacro:imu parent="flange" prefix="imu" color_gazebo="Red">
-        <origin xyz="10 0 0" rpy="0 0 0" />
+        <origin xyz="0.01 0 0" rpy="0 0 0" />
         <color_rgb_rviz>
             <material name="red">
